File: Assignment 2/Assignment 2.kicad_sch (KiCad schematic)
At the start: 45 parts, among them J1 Conn_01x03_Socket, J2 Conn_01x03_Pin, SW1 SW_Push, SW2 SW_Push, U1 AP2112K-3.3, U2 ESP32-S3-WROOM, U3 AL8860MP, U4 AL8860MP, U5 TPS54202DDC, U6 AL8860MP

Commit message: help
Parts:
- added J3: USB-C Plug, Library:GCT_USB4085-GF-A_REVB, symbol Connector:USB_C_Receptacle_PowerOnly_6P
- added R13: 10K, symbol Device:R_Small
- D1, D11, D3: footprint (none) -> LED_SMD:LED_RGB_Getian_GT-P6PRGB4303; MPN (none) -> GT-P6PRGB4303
- D10, D2, D7: value D0V7 -> D0.7V; footprint (none) -> LED_SMD:LED_0603_1608Metric; MPN (none) -> LTW-C191DS5
- J1, J2: footprint (none) -> Connector_PinHeader_1.00mm:PinHeader_1x03_P1.00mm_Vertical; MPN (none) -> B3B-XH-A
- L1, L2, L3: footprint (none) -> Library:INDC1608X100N; MPN (none) -> CBMF1608T470K
- L4: renamed from 15uH; value L -> 15uH; footprint (none) -> Library:INDC2012X145N; MPN (none) -> MLZ2012M150WT000
- R1, R10, R12: value R066 -> 100R
- R5: value 49R9 -> 49.9R
- R7: value 13R3K -> 13.3K
- SW1, SW2: footprint (none) -> Button_Switch_SMD:SW_Push_1P1T_NO_CK_KSC7xxJ; MPN (none) -> D6C90 F2 LFS
- U1: MPN (none) -> AP2112K-3.3
- U2: footprint Library:XCVR_ESP32-S3-WROOM-1-N4 -> RF_Module:ESP32-S2-WROVER; MPN (none) -> ESP32-S3-WROOM
- U3, U4, U6: MPN (none) -> AL8860MP
- U5: MPN (none) -> TPS54202DDC
Connections:
- net +9V: now also J3.A9 (VBUS), J3.B9 (VBUS)
- net GND: now also J3.A12 (GND), J3.B12 (GND), R13.1
- net at U2.22 (USB_D-): now also J3.A5 (CC1)
- net at U2.23 (USB_D+): now also J3.B5 (CC2)
- new net: J3.S1 (SHIELD), R13.2

Commit message: kelp
Parts:
- removed D11: LED B3V1A, LED_SMD:LED_RGB_Getian_GT-P6PRGB4303, symbol Device:LED
- removed D3: LED G3V1A, LED_SMD:LED_RGB_Getian_GT-P6PRGB4303, symbol Device:LED
- removed J3: USB-C Plug, Library:GCT_USB4085-GF-A_REVB, symbol Connector:USB_C_Receptacle_PowerOnly_6P
- added C14: 1uF, symbol Device:C
- added D4: LED_RGB_EP, Diode_SMD:D_0603_1608Metric, symbol Device:LED_RGB_EP
- added D5, D6: D_Small, symbol Device:D_Small
- added J3: USB_C_Receptacle_USB2.0_16P, Library:USB_C_Receptacle_GCT_USB4085, symbol Connector:USB_C_Receptacle_USB2.0_16P
- added R14: 300R, symbol Device:R_Small
- D10, D2, D7: footprint LED_SMD:LED_0603_1608Metric -> Diode_SMD:D_0603_1608Metric; MPN LTW-C191DS5 -> RB070MM-30TFTR
- L1, L2, L3: MPN CBMF1608T470K -> PA4302.473NLT
- L4: MPN MLZ2012M150WT000 -> SRR1208-150ML
- R1, R10, R12: value 100R -> 1R
- U2: footprint RF_Module:ESP32-S2-WROVER -> Library:XCVR_ESP32-S3-WROOM-1-N4
Connections:
- net 5V, 2A: now also D6.2 (A); no longer U1.1 (VIN), U1.3 (EN)
- net GND: now also C14.1
- net at R8.1: now also J2.1 (Pin_1); no longer J2.2 (Pin_2)
- net +3.3V: now reaches R2.1, U1.5 (VOUT), U2.2 (3V3)
- net +3.3V: now also C14.2
- net at C10.1, R9.2, U4.4 (CTRL): now also R14.2
- net 3V1A: now reaches L1.1
- net 3V1A: now also L3.1
- net at R9.1: now also J2.3 (Pin_3); no longer J2.1 (Pin_1)
- net at R11.1: now also J2.2 (Pin_2); no longer J2.3 (Pin_3)
- new net: D5.1 (K), D6.1 (K), U1.1 (VIN), U1.3 (EN)
- new net: J3.A1 (GND), J3.A12 (GND), J3.B1 (GND), J3.B12 (GND)
- new net: J3.A4 (VBUS), J3.A9 (VBUS), J3.B4 (VBUS), J3.B9 (VBUS)
- new net VUSB: D5.2 (A)
Other:
- moved on the sheet: C1, C10, C11, C12, C13, C9, D1, D10, D2, D7, J2, L1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
