File: Assignment 2/Assignment 2.kicad_sch (KiCad schematic)
At the start: 50 parts, among them J3 USB_C_Receptacle_USB2.0_16P, SW1 SW_Push, SW2 SW_Push, U1 AP2112K-3.3, U2 ESP32-S3-WROOM, U3 AL8860MP, U4 AL8860MP, U5 TPS54202DDC, U6 AL8860MP

Commit message: ...
its joever
Parts:
- D10, D2, D5, D6, D7: footprint Library:SODFL3617X108N -> Diode_SMD:D_SOD-123F
- L1, L2, L3: footprint Library:INDC1608X100N -> Inductor_SMD:L_7.3x7.3_H4.5
- L4: footprint Library:INDC2012X145N -> Inductor_SMD:L_Bourns_SRR1208_12.7x12.7mm
Changed lines of the file:
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@@
       (effects (font (size 1.27 1.27)) (justify left))
     )
-    (property "Footprint" "Library:INDC1608X100N" (at 97.79 190.5 0)
+    (property "Footprint" "Inductor_SMD:L_7.3x7.3_H4.5" (at 97.79 190.5 0)
       (effects (font (size 1.27 1.27)) hide)
     )
@@
       (effects (font (size 1.27 1.27)) (justify left))
     )
-    (property "Footprint" "Library:SODFL3617X108N" (at 111.76 133.35 0)
+    (property "Footprint" "Diode_SMD:D_SOD-123F" (at 111.76 133.35 0)
       (effects (font (size 1.27 1.27)) hide)
     )
@@
       (effects (font (size 1.27 1.27)) (justify left))
     )
-    (property "Footprint" "Library:INDC1608X100N" (at 97.79 146.05 0)
+    (property "Footprint" "Inductor_SMD:L_7.3x7.3_H4.5" (at 97.79 146.05 0)
       (effects (font (size 1.27 1.27)) hide)
     )
@@
       (effects (font (size 1.27 1.27)))
     )
-    (property "Footprint" "Library:INDC2012X145N" (at 73.66 35.56 0)
+    (property "Footprint" "Inductor_SMD:L_Bourns_SRR1208_12.7x12.7mm" (at 73.66 35.56 0)
       (effects (font (size 1.27 1.27)) hide)
     )
@@
       (effects (font (size 1.27 1.27)) (justify left))
     )
-    (property "Footprint" "Library:SODFL3617X108N" (at 109.22 179.07 0)
+    (property "Footprint" "Diode_SMD:D_SOD-123F" (at 109.22 179.07 0)
       (effects (font (size 1.27 1.27)) hide)
     )
@@
       (effects (font (size 1.27 1.27)) (justify right))
     )
-    (property "Footprint" "Library:SODFL3617X108N" (at 115.57 33.02 90)
+    (property "Footprint" "Diode_SMD:D_SOD-123F" (at 115.57 33.02 90)
       (effects (font (size 1.27 1.27)) hide)
     )
@@
       (effects (font (size 1.27 1.27)) (justify left))
     )
-    (property "Footprint" "Library:INDC1608X100N" (at 99.06 102.87 0)
+    (property "Footprint" "Inductor_SMD:L_7.3x7.3_H4.5" (at 99.06 102.87 0)
       (effects (font (size 1.27 1.27)) hide)
     )
@@
       (effects (font (size 1.27 1.27)))
     )
-    (property "Footprint" "Library:SODFL3617X108N" (at 110.49 35.56 90)
+    (property "Footprint" "Diode_SMD:D_SOD-123F" (at 110.49 35.56 90)
       (effects (font (size 1.27 1.27)) hide)
     )
@@
       (effects (font (size 1.27 1.27)) (justify left))
     )
-    (property "Footprint" "Library:SODFL3617X108N" (at 113.03 95.25 0)
-      (effects (font (size 1.27 1.27)) hide)
-    )
+    (property "Footprint" "Diode_SMD:D_SOD-123F" (at 113.03 95.25 0)
+      (effects (font (size 1.27 1.27)) hide)
+    )

Commit message: bop
ssd
Parts:
- added BT1: Battery, Battery:BatteryHolder_MPD_BA9VPC_1xPP3, symbol Device:Battery
- U2: footprint Library:XCVR_ESP32-S3-WROOM-1-N4 -> ESP32-S3-WROOM-1-N4:XCVR_ESP32-S3-WROOM-1-N4; symbol RF_Module:ESP32-S2-WROVER -> RF_Module:ESP32-S3-WROOM-1-N4; Availability (none) -> In Stock; Check_prices (none) -> https://www.snapeda.com/parts/ESP32-S3-WROOM-1-N4/Espressif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; MANUFACTURER (none) -> Espressif; MAXIMUM_PACKAGE_HEIGHT (none) -> 3.25mm; MF (none) -> Espressif Systems; MP (none) -> ESP32-S3-WROOM-1-N4; PARTREV (none) -> v1.0; Package (none) -> NON STANDARD Espressif Systems; Price (none) -> None; Purchase-URL (none) -> https://www.snapeda.com/api/url_track_click_mouser/?unipart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; STANDARD (none) -> Manufacturer Recommendations; SnapEDA_Link (none) -> https://www.snapeda.com/parts/ESP32-S3-WROOM-1-N4/Espressif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
Connections:
- net +9V: now also BT1.1 (+)
- net BOOT: now also U2.27 (IO0); no longer U2.3 (IO00)
- net DATA1: now also U2.29 (IO36); no longer U2.36 (IO42)
- net DATA2: now also U2.30 (IO37); no longer U2.35 (IO41)
- net DATA3: now also U2.31 (IO38); no longer U2.34 (IO40)
- net GND: now also U2.40 (GND), U2.41_1 (GND), U2.41_2 (GND), U2.41_3 (GND), U2.41_4 (GND), U2.41_5 (GND), U2.41_6 (GND), U2.41_7 (GND), U2.41_8 (GND), U2.41_9 (GND), BT1.2 (-); no longer U2.26 (GND), U2.42 (GND), U2.43 (GND)
- net at C3.2, R2.2, SW1.2: now also U2.3 (EN); no longer U2.41 (EN)
- net at U2.13 (IO19): now also J3.A7 (D-), J3.B7 (D-)
- net at U2.14 (IO20): now also J3.A6 (D+), J3.B6 (D+)
- now unconnected: U2.22 (USB_D-), U2.23 (USB_D+)
Other:
- moved on the sheet: C14, J3, R13, R15

Commit message: new
Parts:
- U2: footprint ESP32-S3-WROOM-1-N4:XCVR_ESP32-S3-WROOM-1-N4 -> RF_Module:ESP32-S3-WROOM-1
Connections:
- net DATA1: now also U2.31 (IO38); no longer U2.29 (IO36)
- net DATA3: now also U2.29 (IO36); no longer U2.31 (IO38)
- net GND: now also U2.41 (GND); no longer U2.41_1 (GND)
Changed lines of the file:
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@@
-    (stroke (width 0) (type default))
-  )
-  (wire (pts (xy 212.09 58.42) (xy 209.55 58.42))
     (stroke (width 0) (type default))
   )
@@
   )
   (wire (pts (xy 100.33 44.45) (xy 100.33 43.18))
-    (stroke (width 0) (type default))
-  )
-  (wire (pts (xy 212.09 63.5) (xy 209.55 63.5))
     (stroke (width 0) (type default))
   )
@@
     (effects (font (size 1.27 1.27)) (justify left bottom))
   )
-  (label "DATA1" (at 212.09 58.42 0) (fields_autoplaced)
+  (label "DATA1" (at 209.55 63.5 0) (fields_autoplaced)
     (effects (font (size 1.27 1.27)) (justify left bottom))
   )
@@
     (effects (font (size 1.27 1.27)) (justify left bottom))
   )
-  (label "DATA3" (at 212.09 63.5 0) (fields_autoplaced)
+  (label "DATA3" (at 209.55 58.42 0) (fields_autoplaced)
     (effects (font (size 1.27 1.27)) (justify left bottom))
   )
@@
       (effects (font (size 1.27 1.27)))
     )
-    (property "Footprint" "ESP32-S3-WROOM-1-N4:XCVR_ESP32-S3-WROOM-1-N4" (at 194.31 58.42 0)
+    (property "Footprint" "RF_Module:ESP32-S3-WROOM-1" (at 194.31 58.42 0)
       (effects (font (size 1.27 1.27)) (justify bottom) hide)
     )
@@
     (pin "21")
     (pin "22")
-    (pin "41_1")
+    (pin "41")
     (pin "41_2")
     (pin "40")

Commit message: sdsjd
Parts:
- C8: value 75pF -> 100pF
Changed lines of the file:
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@@
       (effects (font (size 1.27 1.27)) (justify right))
     )
-    (property "Value" "75pF" (at 99.06 46.99 0)
+    (property "Value" "100pF" (at 99.06 46.99 0)
       (effects (font (size 1.27 1.27)) (justify right))
     )
