File: Assignment 2/Assignment 2.kicad_pcb (KiCad board)
At the start: 4 copper layers, 0 parts

Commit message: null
Parts:
- added C1: 10uF, Capacitor_SMD:C_1206_3216Metric, F.Cu at (140.2, 52.3)
- added C10: 10nF, Capacitor_SMD:C_0603_1608Metric, F.Cu at (134.9, 83.3)
- added C11: 10uF, Capacitor_SMD:C_1206_3216Metric, F.Cu at (140.6, 78.3)
- added C12: 10nF, Capacitor_SMD:C_0603_1608Metric, F.Cu at (135.0, 70.3)
- added C13: 10uF, Capacitor_SMD:C_1206_3216Metric, F.Cu at (140.3, 65.3)
- added C14: 1uF, Capacitor_SMD:C_0603_1608Metric, F.Cu at (124.8, 48.0)
- added C2: 10uF, Capacitor_SMD:C_1206_3216Metric, F.Cu at (94.5, 40.0)
- added C3: 1uF, Capacitor_SMD:C_0603_1608Metric, F.Cu at (124.8, 45.0)
- added C4: 0.1uF, Capacitor_SMD:C_0603_1608Metric, F.Cu at (94.0, 45.0)
- added C5: 0.1uF, Capacitor_SMD:C_0603_1608Metric, F.Cu at (110.0, 41.8)
- added C6: 22uF, Capacitor_SMD:C_0603_1608Metric, F.Cu at (114.0, 41.5)
- added C7: 22uF, Capacitor_SMD:C_0603_1608Metric, F.Cu at (114.0, 45.2)
- added C8: 75pF, Capacitor_SMD:C_0603_1608Metric, F.Cu at (103.9, 49.9)
- added C9: 10nF, Capacitor_SMD:C_0603_1608Metric, F.Cu at (135.0, 57.3)
- added D10: RB070mm, Library:SODFL3617X108N, F.Cu at (150.3, 53.3)
- added D2: RB070mm, Library:SODFL3617X108N, F.Cu at (151.3, 79.3)
- added D4: LED_RGB_EP, LED_SMD:LED_RGB_Getian_GT-P6PRGB4303, F.Cu at (144.2, 44.7)
- added D5: RB070mm, Library:SODFL3617X108N, F.Cu at (119.5, 41.0)
- added D6: RB070mm, Library:SODFL3617X108N, F.Cu at (119.0, 45.0)
- added D7: RB070mm, Library:SODFL3617X108N, F.Cu at (150.3, 66.3)
- added J3: USB_C_Receptacle_USB2.0_16P, Library:USB_C_Receptacle_GCT_USB4085, F.Cu at (100.0, 72.8)
- added L1: 47uH, Library:INDC1608X100N, F.Cu at (150.8, 56.3)
- added L2: 47uH, Library:INDC1608X100N, F.Cu at (150.8, 82.3)
- added L3: 47uH, Library:INDC1608X100N, F.Cu at (150.5, 69.3)
- added L4: 15uH, Library:INDC2012X145N, F.Cu at (110.0, 45.9)
- added R1: 1R, Resistor_SMD:R_0603_1608Metric, F.Cu at (145.8, 52.1)
- added R10: 1R, Resistor_SMD:R_0603_1608Metric, F.Cu at (146.1, 78.4)
- added R11: 300R, Resistor_SMD:R_0603_1608Metric, F.Cu at (134.9, 65.3)
- added R12: 1R, Resistor_SMD:R_0603_1608Metric, F.Cu at (145.8, 65.3)
- added R13: 5.1K, Resistor_SMD:R_0603_1608Metric, F.Cu at (100.0, 54.9)
- added R14: 10K, Resistor_SMD:R_0603_1608Metric, F.Cu at (139.9, 83.3)
- added R15: 5.1K, Resistor_SMD:R_0603_1608Metric, F.Cu at (100.0, 59.9)
- added R16: 10K, Resistor_SMD:R_0603_1608Metric, F.Cu at (139.9, 70.3)
- added R17: 10K, Resistor_SMD:R_0603_1608Metric, F.Cu at (139.6, 57.3)
- added R2: 10K, Resistor_SMD:R_0603_1608Metric, F.Cu at (124.7, 42.0)
- added R3: 511K, Resistor_SMD:R_0603_1608Metric, F.Cu at (99.8, 40.2)
- added R4: 105K, Resistor_SMD:R_0603_1608Metric, F.Cu at (100.2, 45.0)
- added R5: 49.9R, Resistor_SMD:R_0603_1608Metric, F.Cu at (109.9, 49.7)
- added R6: 100K, Resistor_SMD:R_0603_1608Metric, F.Cu at (106.9, 49.7)
- added R7: 13.3K, Resistor_SMD:R_0603_1608Metric, F.Cu at (100.9, 49.9)
- added R8: 300R, Resistor_SMD:R_0603_1608Metric, F.Cu at (134.9, 52.3)
- added R9: 300R, Resistor_SMD:R_0603_1608Metric, F.Cu at (134.9, 78.3)
- added SW1: SW_Push, Button_Switch_SMD:SW_Push_1P1T_NO_CK_KSC7xxJ, F.Cu at (108.0, 57.1)
- added SW2: SW_Push, Button_Switch_SMD:SW_Push_1P1T_NO_CK_KSC7xxJ, F.Cu at (119.0, 57.1)
- added U1: AP2112K-3.3, Package_TO_SOT_SMD:SOT-23-5, F.Cu at (119.1, 49.0)
- added U2: ESP32-S3-WROOM, Library:XCVR_ESP32-S3-WROOM-1-N4, F.Cu at (118.9, 76.8)
- added U3: AL8860MP, Package_SO:MSOP-8-1EP_3x3mm_P0.65mm_EP1.5x1.8mm, F.Cu at (145.1, 58.0)
- added U4: AL8860MP, Package_SO:MSOP-8-1EP_3x3mm_P0.65mm_EP1.5x1.8mm, F.Cu at (145.2, 84.9)
- added U5: TPS54202DDC, Package_TO_SOT_SMD:SOT-23-6, F.Cu at (105.0, 42.1)
- added U6: AL8860MP, Package_SO:MSOP-8-1EP_3x3mm_P0.65mm_EP1.5x1.8mm, F.Cu at (145.3, 70.9)
Routing:
- net GND: track 0.00 -> 207.9 mm, vias 0 -> 2
- net /RED_IN: track 0.00 -> 50.9 mm, vias 0 -> 3
- net +9V: track 0.00 -> 48.8 mm
- net /DATA1: track 0.00 -> 46.6 mm, vias 0 -> 2
- net /DATA2: track 0.00 -> 42.9 mm, vias 0 -> 3
- net /RED_OUT: track 0.00 -> 39.4 mm, vias 0 -> 2
- net /GREEN_IN: track 0.00 -> 37.9 mm, vias 0 -> 3
- net Net-(U2-EN): track 0.00 -> 36.7 mm, vias 0 -> 3
- net /BLUE_IN: track 0.00 -> 32.5 mm, vias 0 -> 2
- net +3.3V: track 0.00 -> 32.0 mm, vias 0 -> 2
- net /GREEN_OUT: track 0.00 -> 30.0 mm, vias 0 -> 2
- net /DATA3: track 0.00 -> 28.9 mm
- net Net-(U4-CTRL): track 0.00 -> 21.8 mm
- net Net-(J3-CC1): track 0.00 -> 21.5 mm
- net Net-(U6-CTRL): track 0.00 -> 20.8 mm
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Other:
- copper layers 4 -> 2

Commit message: ...
its joever
Parts:
- D10, D2, D5, D6, D7: footprint Library:SODFL3617X108N -> Diode_SMD:D_SOD-123F
- L1, L2, L3: footprint Library:INDC1608X100N -> Inductor_SMD:L_7.3x7.3_H4.5
- L4: footprint Library:INDC2012X145N -> Inductor_SMD:L_Bourns_SRR1208_12.7x12.7mm
- moved D4 88.5 mm to (105.0, 124.0)
- moved L2 68.5 mm to (89.0, 111.8), turned to 90 degrees
- moved L1 64.7 mm to (117.6, 111.8), turned to 90 degrees
- moved L3 63.8 mm to (103.0, 111.8), turned to 90 degrees
- moved D2 61.8 mm to (94.0, 102.4), turned to -90 degrees
- moved R10 61.1 mm to (87.8, 97.0), turned to 180 degrees
- moved U4 59.5 mm to (88.4, 102.5), turned to 0 degrees
- moved D10 56.7 mm to (122.0, 102.4), turned to -90 degrees
- moved D7 55.6 mm to (108.0, 102.4), turned to -90 degrees
- moved R12 54.7 mm to (101.2, 97.0), turned to 180 degrees
- moved R1 54.4 mm to (115.0, 97.0), turned to 180 degrees
- moved U6 53.9 mm to (101.9, 102.7), turned to 0 degrees
- moved U3 53.5 mm to (115.4, 102.5), turned to 0 degrees
- moved R14 52.8 mm to (88.0, 92.8), turned to -90 degrees
- moved C11 49.0 mm to (94.0, 93.5), turned to 90 degrees
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Routing:
- net +9V: track 48.8 -> 153.2 mm, vias 0 -> 9
- net GND: track 207.9 -> 292.7 mm, vias 2 -> 20
- net /DATA1: track 46.6 -> 6.95 mm, vias 2 -> 0
- net /5V, 2A: track 16.1 -> 48.6 mm, vias 2 -> 0
- net Net-(D5-K): track 3.47 -> 30.4 mm, vias 0 -> 2
- net /DATA2: track 42.9 -> 19.7 mm, vias 3 -> 0
- net Net-(U2-USB_D+): track 0.00 -> 22.2 mm, vias 0 -> 1
- net Net-(U2-USB_D-): track 0.00 -> 20.8 mm, vias 0 -> 1
- net Net-(J3-CC2): track 20.6 -> 0.00 mm
- net +3.3V: track 32.0 -> 46.6 mm
- net /BLUE_IN: track 32.5 -> 46.9 mm, vias 2 -> 7
- net Net-(J3-CC1): track 21.5 -> 8.46 mm
- net Net-(U5-SW): track 10.9 -> 22.1 mm
- net /BOOT: track 15.7 -> 26.2 mm
- net /RED_IN: track 50.9 -> 42.8 mm, vias 3 -> 2
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Other:
- board text added: "Buck Convertor - B"
- board text added: "Buck Convertor - G"
- board text added: "Buck Convertor - R"
- board text added: "ESP32 and USBC"
- board text added: "LED"
- board text added: "Regulator"
- board text added: "Step Down Converter"

Commit message: sob
sdkjsjd
Routing:
- net GND: track 292.7 -> 294.2 mm
Changed lines of the file:
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@@
   (segment (start 112 33) (end 118.35 33) (width 0.2) (layer "F.Cu") (net 2))
   (segment (start 121 60) (end 124.61 63.61) (width 0.2) (layer "F.Cu") (net 2))
+  (segment (start 101.750735 95.249265) (end 104 93) (width 0.2) (layer "F.Cu") (net 2))
   (segment (start 94.45 88.55) (end 94 88.55) (width 0.2) (layer "F.Cu") (net 2))
   (segment (start 115.375 102.55) (end 113.5875 102.55) (width 0.2) (layer "F.Cu") (net 2))
@@
   (segment (start 96 47) (end 96.6 46.4) (width 0.2) (layer "F.Cu") (net 2))
   (segment (start 117 37.05) (end 117 35) (width 0.2) (layer "F.Cu") (net 2))
+  (segment (start 118 92) (end 115 95) (width 0.2) (layer "F.Cu") (net 2))
   (segment (start 113.725 53) (end 107.8 53) (width 0.2) (layer "F.Cu") (net 2))
   (segment (start 102 105) (end 101.8875 104.8875) (width 0.2) (layer "F.Cu") (net 2))
@@
   (segment (start 90 49.775) (end 94.775 49.775) (width 0.2) (layer "F.Cu") (net 2))
   (segment (start 121 92) (end 115 92) (width 0.2) (layer "F.Cu") (net 2))
-  (segment (start 94 92) (end 88 92) (width 0.2) (layer "F.Cu") (net 2))
+  (segment (start 88 95) (end 89 95) (width 0.2) (layer "F.Cu") (net 2))
   (segment (start 101.8875 102.730956) (end 101.8875 102.1125) (width 0.2) (layer "F.Cu") (net 2))
+  (segment (start 89 95) (end 91 93) (width 0.2) (layer "F.Cu") (net 2))
   (segment (start 88 105) (end 88.375 104.625) (width 0.2) (layer "F.Cu") (net 2))
   (segment (start 94.775 49.775) (end 96 48.55) (width 0.2) (layer "F.Cu") (net 2))
@@
   (segment (start 88.375 102.45) (end 88.375 101.375) (width 0.2) (layer "F.Cu") (net 2))
   (segment (start 100.19054 41.80946) (end 104 38) (width 0.2) (layer "F.Cu") (net 2))
+  (segment (start 101 92) (end 104 92) (width 0.2) (layer "F.Cu") (net 2))
+  (segment (start 104 93) (end 104 92) (width 0.2) (layer "F.Cu") (net 2))
   (segment (start 115.375 102.55) (end 115.375 101.375) (width 0.2) (layer "F.Cu") (net 2))
   (segment (start 96.6 82) (end 96.6 83.4) (width 0.2) (layer "F.Cu") (net 2))
@@
   (segment (start 113.725 53) (end 120.225 53) (width 0.2) (layer "F.Cu") (net 2))
   (segment (start 99.775 102.405956) (end 99.775 103.055956) (width 0.2) (layer "F.Cu") (net 2))
+  (segment (start 100.249265 95.249265) (end 101.750735 95.249265) (width 0.2) (layer "F.Cu") (net 2))
   (segment (start 113.2625 102.875) (end 113.2625 102.225) (width 0.2) (layer "F.Cu") (net 2))
   (segment (start 96.6 83.4) (end 96 84) (width 0.2) (layer "F.Cu") (net 2))
@@
   (segment (start 115.375 102.55) (end 115.375 103.65) (width 0.2) (layer "F.Cu") (net 2))
   (segment (start 102 105) (end 90 105) (width 0.2) (layer "F.Cu") (net 2))
+  (segment (start 91 93) (end 91 92) (width 0.2) (layer "F.Cu") (net 2))
+  (segment (start 94 92) (end 91 92) (width 0.2) (layer "F.Cu") (net 2))
   (segment (start 88.225 49.775) (end 87.1 50.9) (width 0.2) (layer "F.Cu") (net 2))
+  (segment (start 91 92) (end 88 92) (width 0.2) (layer "F.Cu") (net 2))
   (segment (start 100.22961 46.336075) (end 100.22961 46.554329) (width 0.2) (layer "F.Cu") (net 2))
   (segment (start 121 53.775) (end 121 60) (width 0.2) (layer "F.Cu") (net 2))
   (segment (start 92.15 77.55) (end 88.025 77.55) (width 0.2) (layer "F.Cu") (net 2))
   (segment (start 83.665 52.335) (end 84 52) (width 0.2) (layer "F.Cu") (net 2))
-  (segment (start 101 92) (end 107 92) (width 0.2) (layer "F.Cu") (net 2))
+  (segment (start 104 92) (end 107 92) (width 0.2) (layer "F.Cu") (net 2))
   (segment (start 83.665 70.25) (end 83.665 52.335) (width 0.2) (layer "F.Cu") (net 2))
   (segment (start 86.2625 102.125) (end 88.05 102.125) (width 0.2) (layer "F.Cu") (net 2))
   (segment (start 100.1 102.730956) (end 99.775 102.405956) (width 0.2) (layer "F.Cu") (net 2))
   (via (at 117 35) (size 0.6) (drill 0.3) (layers "F.Cu" "B.Cu") (net 2))
-  (via (at 118 92) (size 0.6) (drill 0.3) (layers "F.Cu" "B.Cu") (net 2))
   (via (at 100 100) (size 0.6) (drill 0.3) (layers "F.Cu" "B.Cu") (net 2))
   (via (at 100.22961 46.554329) (size 0.6) (drill 0.3) (layers "F.Cu" "B.Cu") (net 2))
   (via (at 100.19054 44.96093) (size 0.6) (drill 0.3) (layers "F.Cu" "B.Cu") (net 2))
   (via (at 96 84) (size 0.6) (drill 0.3) (layers "F.Cu" "B.Cu") (net 2))
-  (via (at 91 92) (size 0.6) (drill 0.3) (layers "F.Cu" "B.Cu") (net 2))
   (via (at 115 33) (size 0.6) (drill 0.3) (layers "F.Cu" "B.Cu") (net 2))
   (via (at 90 105) (size 0.6) (drill 0.3) (layers "F.Cu" "B.Cu") (net 2))
@@
   (via (at 102 105) (size 0.6) (drill 0.3) (layers "F.Cu" "B.Cu") (net 2))
   (via (at 90 105) (size 0.6) (drill 0.3) (layers "F.Cu" "B.Cu") (net 2))
+  (via (at 88 95) (size 0.6) (drill 0.3) (layers "F.Cu" "B.Cu") (net 2))
   (via (at 87 100) (size 0.6) (drill 0.3) (layers "F.Cu" "B.Cu") (net 2))
   (via (at 88 105) (size 0.6) (drill 0.3) (layers "F.Cu" "B.Cu") (net 2))
@@
   (via (at 106 38) (size 0.6) (drill 0.3) (layers "F.Cu" "B.Cu") (net 2))
   (via (at 87.1 52) (size 0.6) (drill 0.3) (layers "F.Cu" "B.Cu") (net 2))
+  (via (at 100.249265 95.249265) (size 0.6) (drill 0.3) (layers "F.Cu" "B.Cu") (net 2))
+  (via (at 115 95) (size 0.6) (drill 0.3) (layers "F.Cu" "B.Cu") (net 2))
   (via (at 104 105) (size 0.6) (drill 0.3) (layers "F.Cu" "B.Cu") (net 2))
-  (via (at 104 92) (size 0.6) (drill 0.3) (layers "F.Cu" "B.Cu") (net 2))
   (segment (start 85.6 72.180026) (end 85.6 76.68566) (width 0.2) (layer "B.Cu") (net 2))
   (segment (start 116 34) (end 110 34) (width 0.2) (layer "B.Cu") (net 2))
   (segment (start 86.675 77.55) (end 88.025 77.55) (width 0.2) (layer "B.Cu") (net 2))
   (segment (start 86.675 71.6) (end 86.180026 71.6) (width 0.2) (layer "B.Cu") (net 2))
+  (segment (start 100 95.49853) (end 100.249265 95.249265) (width 0.2) (layer "B.Cu") (net 2))
   (segment (start 86.675 71.6) (end 88.025 71.6) (width 0.2) (layer "B.Cu") (net 2))
   (segment (start 110 34) (end 106 38) (width 0.2) (layer "B.Cu") (net 2))
@@
   (segment (start 85.6 76.68566) (end 86.46434 77.55) (width 0.2) (layer "B.Cu") (net 2))
   (segment (start 100.22961 46.554329) (end 100.22961 45) (width 0.2) (layer "B.Cu") (net 2))
+  (segment (start 115 95) (end 114 96) (width 0.2) (layer "B.Cu") (net 2))
+  (segment (start 100 96) (end 100 95.49853) (width 0.2) (layer "B.Cu") (net 2))
   (segment (start 116 34) (end 115 33) (width 0.2) (layer "B.Cu") (net 2))
   (segment (start 117 35) (end 116 34) (width 0.2) (layer "B.Cu") (net 2))
@@
   (segment (start 100.22961 45) (end 100.19054 44.96093) (width 0.2) (layer "B.Cu") (net 2))
   (segment (start 96 84) (end 96 86) (width 0.2) (layer "B.Cu") (net 2))
-  (segment (start 114 96) (end 118 92) (width 0.2) (layer "B.Cu") (net 2))
-  (segment (start 87 96) (end 91 92) (width 0.2) (layer "B.Cu") (net 2))
   (segment (start 87.045 71.23) (end 86.675 71.6) (width 0.2) (layer "B.Cu") (net 2))
   (segment (start 104 105) (end 102 105) (width 0.2) (layer "B.Cu") (net 2))
@@
   (segment (start 87.045 70.25) (end 87.045 71.23) (width 0.2) (layer "B.Cu") (net 2))
   (segment (start 83.665 78.9) (end 87.045 78.9) (width 0.2) (layer "B.Cu") (net 2))
-  (segment (start 100 96) (end 104 92) (width 0.2) (layer "B.Cu") (net 2))
+  (segment (start 87 96) (end 88 95) (width 0.2) (layer "B.Cu") (net 2))
   (segment (start 90 105) (end 88 105) (width 0.2) (layer "B.Cu") (net 2))
   (segment (start 100 100) (end 100 96) (width 0.2) (layer "B.Cu") (net 2))

Commit message: bop
ssd
Parts:
- added BT1: Battery, Battery:BatteryHolder_MPD_BA9VPC_1xPP3, F.Cu at (230.1, 77.0)
- moved C5 155.6 mm to (235.2, 117.0), turned to 180 degrees
- moved R7 155.3 mm to (241.8, 117.0)
- moved C4 154.5 mm to (241.0, 110.2), turned to 90 degrees
- moved R4 153.9 mm to (248.2, 117.0)
- moved C2 148.6 mm to (247.0, 110.5), turned to 90 degrees
- moved L4 148.2 mm to (222.0, 112.0), turned to 90 degrees
- moved U5 143.7 mm to (234.9, 110.0), turned to 180 degrees
- moved C8 143.3 mm to (249.0, 100.0), turned to -90 degrees
- moved R3 142.2 mm to (247.8, 105.0), turned to 0 degrees
- moved SW1 141.8 mm to (228.1, 89.0), turned to 180 degrees
- moved R6 140.6 mm to (241.0, 100.0), turned to -90 degrees
- moved R5 140.2 mm to (233.2, 100.0)
- moved R9 140.2 mm to (215.3, 29.0), turned to 180 degrees
- moved C7 139.8 mm to (225.0, 99.8), turned to 90 degrees
- moved C6 138.6 mm to (219.0, 99.8), turned to 90 degrees
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Connections:
- J3 pad A6: Net-(U2-USB_D+) -> Net-(U2-IO20)
- J3 pad A7: Net-(U2-USB_D-) -> Net-(U2-IO19)
- J3 pad B6: Net-(U2-USB_D+) -> Net-(U2-IO20)
- J3 pad B7: Net-(U2-USB_D-) -> Net-(U2-IO19)
Routing:
- net GND: track 294.2 -> 365.1 mm, vias 20 -> 16
- net /DATA3: track 31.4 -> 91.5 mm
- net /DATA2: track 19.7 -> 73.6 mm
- net /DATA1: track 6.95 -> 55.3 mm
- net +3.3V: track 46.6 -> 92.0 mm, vias 2 -> 4
- net +9V: track 153.2 -> 181.7 mm, vias 9 -> 6
- net Net-(D5-K): track 30.4 -> 57.9 mm, vias 2 -> 5
- net /BOOT: track 26.2 -> 48.8 mm
- net Net-(U2-USB_D+): track 22.2 -> 0.00 mm, vias 1 -> 0
- net Net-(U2-USB_D-): track 20.8 -> 0.00 mm, vias 1 -> 0
- net Net-(U5-FB): track 18.6 -> 36.8 mm, vias 4 -> 0
- net /5V, 2A: track 48.6 -> 31.6 mm
- net Net-(U2-EN): track 36.4 -> 23.6 mm
- net Net-(U5-EN): track 17.9 -> 30.3 mm
- net Net-(U4-CTRL): track 24.2 -> 14.6 mm
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- added copper zone on F.Cu, net +9V
- added copper zone on F.Cu, net GND
Other:
- board outline added: 81.2 x 99.2 mm

Commit message: new
Parts:
- U2: footprint Library:XCVR_ESP32-S3-WROOM-1-N4 -> RF_Module:ESP32-S3-WROOM-1
- moved R4 17.7 mm to (235.2, 105.0), turned to 0 degrees
- moved R7 12.0 mm to (241.2, 105.0)
- moved C2 7.42 mm to (244.5, 117.5), turned to 180 degrees
- moved SW2 7.00 mm to (205.3, 89.0)
- moved U5 6.36 mm to (241.1, 111.0)
- moved C3 6.18 mm to (246.1, 86.0), turned to 180 degrees
- moved C4 6.08 mm to (247.0, 111.2)
- moved R2 5.93 mm to (240.0, 86.0), turned to 0 degrees
- moved SW1 5.00 mm to (223.1, 89.0)
- moved C9 1.57 mm to (213.8, 74.0)
- moved C5 1.00 mm to (235.2, 118.0)
- moved R3 0.65 mm to (247.2, 105.0)
- moved L1 0.59 mm to (189.7, 70.0)
- moved D4 0.50 mm to (178.0, 53.0)
- turned C14 to 90 degrees
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Connections:
- U2 pad 13: unconnected-(U2-IO10-Pad13) -> Net-(U2-IO19)
- U2 pad 14: unconnected-(U2-IO11-Pad14) -> Net-(U2-IO20)
- U2 pad 22: Net-(U2-USB_D-) -> unconnected-(U2-IO14-Pad22)
- U2 pad 23: Net-(U2-USB_D+) -> unconnected-(U2-IO21-Pad23)
- U2 pad 26: GND -> unconnected-(U2-IO45-Pad26)
- U2 pad 27: unconnected-(U2-IO33-Pad27) -> /BOOT
- U2 pad 29: unconnected-(U2-IO35-Pad29) -> /DATA3
- U2 pad 3: /BOOT -> Net-(U2-EN)
- U2 pad 30: unconnected-(U2-IO36-Pad30) -> /DATA2
- U2 pad 31: unconnected-(U2-IO37-Pad31) -> /DATA1
- U2 pad 34: /DATA3 -> unconnected-(U2-IO41-Pad34)
- U2 pad 35: /DATA2 -> unconnected-(U2-IO42-Pad35)
- U2 pad 36: /DATA1 -> unconnected-(U2-RXD0-Pad36)
- U2 pad 40: unconnected-(U2-IO46-Pad40) -> GND
Routing:
- net GND: track 365.1 -> 0.00 mm, vias 16 -> 0
- net +9V: track 181.7 -> 114.9 mm, vias 6 -> 0
- net Net-(U2-EN): track 23.6 -> 82.0 mm, vias 2 -> 0
- net /5V, 2A: track 31.6 -> 0.00 mm
- net /BOOT: track 48.8 -> 18.5 mm
- net Net-(J3-CC2): track 0.00 -> 19.8 mm, vias 0 -> 2
- net Net-(U5-FB): track 36.8 -> 17.7 mm
- net Net-(U4-CTRL): track 14.6 -> 29.7 mm, vias 0 -> 2
- net Net-(J3-CC1): track 0.00 -> 11.9 mm
- net Net-(U5-EN): track 30.3 -> 21.0 mm
- net /DATA1: track 55.3 -> 46.4 mm, vias 0 -> 2
- net /DATA2: track 73.6 -> 65.9 mm, vias 0 -> 2
- net /GREEN_OUT: track 20.0 -> 13.2 mm, vias 2 -> 0
- net /DATA3: track 91.5 -> 85.1 mm, vias 0 -> 2
- net /RED_IN: track 41.6 -> 47.8 mm
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- added copper zone on F.Cu, net (none)
- added copper zone on F.Cu, net /5V, 2A
- added copper zone on B.Cu, net GND

Commit message: pcbbbb
yayyy???
Parts:
- C8: value 75pF -> 100pF
- moved C3 67.5 mm to (182.9, 109.8)
- moved C14 67.5 mm to (176.0, 116.9)
- moved R2 67.5 mm to (176.9, 109.8)
- moved U1 67.5 mm to (182.9, 116.7)
- moved U2 4.00 mm to (178.4, 91.9)
- moved SW2 1.80 mm to (207.1, 89.0)
- moved SW1 1.00 mm to (224.1, 89.0)
Routing:
- net GND: track 0.00 -> 153.5 mm, vias 0 -> 18
- net +3.3V: track 86.2 -> 22.4 mm
- net /5V, 2A: track 0.00 -> 31.3 mm
- net Net-(U2-IO19): track 1.70 -> 21.4 mm, vias 0 -> 2
- net +9V: track 114.9 -> 133.8 mm
- net Net-(U2-IO20): track 1.70 -> 20.4 mm, vias 0 -> 2
- net Net-(D5-K): track 55.4 -> 39.6 mm, vias 0 -> 2
- net Net-(U2-EN): track 82.0 -> 68.7 mm, vias 0 -> 2
- net /BOOT: track 18.5 -> 21.9 mm
- net /DATA2: track 65.9 -> 64.2 mm
- net /DATA1: track 46.4 -> 44.8 mm
- net Net-(U6-CTRL): track 29.9 -> 31.2 mm
- net /DATA3: track 85.1 -> 83.8 mm
- net /RED_OUT: track 35.2 -> 34.6 mm
