File: Assignment 2/Assignment 2.kicad_pcb (KiCad board)
At the start: 2 copper layers, 81.2 x 99.2 mm, 51 parts, among them J3 USB_C_Receptacle_USB2.0_16P, SW1 SW_Push, SW2 SW_Push, U1 AP2112K-3.3, U2 ESP32-S3-WROOM, U3 AL8860MP, U4 AL8860MP, U5 TPS54202DDC, U6 AL8860MP

Commit message: sdsjd
Other:
- board text added: "B-IN"
- board text added: "B-OUT"
- board text added: "G-IN"
- board text added: "G-OUT"
- board text added: "R-IN"
- board text added: "R-OUT"
- board text added: "VIA - SMART LED"
Changed lines of the file:
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@@
     (property "ki_keywords" "inductor choke coil reactor magnetic")
     (attr smd)
-    (fp_text reference "L2" (at 0 -4.45) (layer "F.SilkS")
-        (effects (font (size 1 1) (thickness 0.15)))
-    )
-    (fp_text value "47uH" (at 0 4.45) (layer "F.Fab")
+    (fp_text reference "L2" (at -2.7 -5) (layer "F.SilkS")
+        (effects (font (size 1 1) (thickness 0.15)))
+    )
+    (fp_text value "47uH" (at 0 5) (layer "F.Fab")
         (effects (font (size 1 1) (thickness 0.15)))
     )
@@
         (effects (font (size 1 1) (thickness 0.15)))
     )
-    (fp_text value "AP2112K-3.3" (at 1.7375 3.1375 90) (layer "F.Fab")
+    (fp_text value "AP2112K-3.3" (at 2.7375 4.1375 90) (layer "F.Fab")
         (effects (font (size 1 1) (thickness 0.15)))
     )
@@
         (effects (font (size 1 1) (thickness 0.15)))
     )
-    (fp_text value "LED_RGB_EP" (at 5.78 -6.7 90) (layer "F.Fab")
+    (fp_text value "LED_RGB_EP" (at 16 -4 90) (layer "F.Fab")
         (effects (font (size 1 1) (thickness 0.15)))
     )
@@
   (gr_rect (start 171.661306 23.062614) (end 252.858694 122.26)
     (stroke (width 0.2) (type default)) (fill none) (layer "Edge.Cuts"))
+  (gr_text "VIA - SMART LED" (at 173 25) (layer "Dwgs.User" knockout)
+    (effects (font (size 0.75 0.75) (thickness 0.125)) (justify left bottom))
+  )
   (gr_text "LED" (at 174 54.575 -90) (layer "Dwgs.User")
     (effects (font (size 0.5 0.5) (thickness 0.125)) (justify left bottom))
   )
-  (gr_text "Buck Convertor - R" (at 185 25) (layer "Dwgs.User")
+  (gr_text "B-IN\n" (at 179 41 90) (layer "Dwgs.User")
     (effects (font (size 0.5 0.5) (thickness 0.125)) (justify left bottom))
   )
-  (gr_text "Regulator" (at 173 121) (layer "Dwgs.User")
+  (gr_text "Buck Convertor - R" (at 185 41) (layer "Dwgs.User" knockout)
     (effects (font (size 0.5 0.5) (thickness 0.125)) (justify left bottom))
   )
-  (gr_text "ESP32 and USBC" (at 203 120) (layer "Dwgs.User")
+  (gr_text "R-IN\n" (at 177 43 90) (layer "Dwgs.User")
     (effects (font (size 0.5 0.5) (thickness 0.125)) (justify left bottom))
   )
-  (gr_text "Buck Convertor - B\n" (at 185 61) (layer "Dwgs.User")
+  (gr_text "Regulator" (at 183 121) (layer "Dwgs.User" knockout)
     (effects (font (size 0.5 0.5) (thickness 0.125)) (justify left bottom))
   )
-  (gr_text "Step Down Converter" (at 243 121) (layer "Dwgs.User")
+  (gr_text "B-OUT\n" (at 181 64 90) (layer "Dwgs.User")
     (effects (font (size 0.5 0.5) (thickness 0.125)) (justify left bottom))
   )
-  (gr_text "Buck Convertor - G" (at 185 44) (layer "Dwgs.User")
+  (gr_text "ESP32 and USBC" (at 206 121) (layer "Dwgs.User" knockout)
+    (effects (font (size 0.5 0.5) (thickness 0.125)) (justify left bottom))
+  )
+  (gr_text "Buck Convertor - B\n" (at 185 62) (layer "Dwgs.User" knockout)
+    (effects (font (size 0.5 0.5) (thickness 0.125)) (justify left bottom))
+  )
+  (gr_text "G-IN\n" (at 178 42 90) (layer "Dwgs.User")
+    (effects (font (size 0.5 0.5) (thickness 0.125)) (justify left bottom))
+  )
+  (gr_text "Step Down Converter" (at 251 120 90) (layer "Dwgs.User" knockout)
+    (effects (font (size 0.5 0.5) (thickness 0.125)) (justify left bottom))
+  )
+  (gr_text "Buck Convertor - G" (at 185 59) (layer "Dwgs.User" knockout)
+    (effects (font (size 0.5 0.5) (thickness 0.125)) (justify left bottom))
+  )
+  (gr_text "R-OUT\n" (at 177 64 90) (layer "Dwgs.User")
+    (effects (font (size 0.5 0.5) (thickness 0.125)) (justify left bottom))
+  )
+  (gr_text "G-OUT\n" (at 179 64 90) (layer "Dwgs.User")
     (effects (font (size 0.5 0.5) (thickness 0.125)) (justify left bottom))
   )
@@
         (xy 248 110)
         (xy 247.281796 106.718204)
-        (xy 247 105)
       )
     )

Commit message: naur
sds
Other:
- board text added: "3V3"
- board text added: "5V, 2A"
- board text added: "9V"
- board text added: "BOOT"
- board text added: "CRTL"
- board text added: "DATA-1"
- board text added: "DATA-2"
- board text added: "DATA-3"
- board text added: "EN"
- board text added: "FB"
- board text added: "GND"
- board text added: "SIG"
- board text added: "SW"
- board text added: "VIA SMART LED"
- board text added: "VUSB"
- board text removed: "VIA - SMART LED"
