File: Assignment 2/Assignment 2.kicad_pcb (KiCad board)
At the start: 2 copper layers, 81.2 x 99.2 mm, 51 parts, among them J3 USB_C_Receptacle_USB2.0_16P, SW1 SW_Push, SW2 SW_Push, U1 AP2112K-3.3, U2 ESP32-S3-WROOM, U3 AL8860MP, U4 AL8860MP, U5 TPS54202DDC, U6 AL8860MP

Commit message: aggg
s
Parts:
- D10, D2, D5, D6, D7: value RB070mm -> RB070
Other:
- board text removed: "LED"

Commit message: irp
asdkjas
Parts:
- added REF**: EdgertonLogo, Library:EdgertonLogo, F.Cu at (173.2, 76.5)
- added REF**: MechELogo, Library:MechELogo, F.Cu at (232.1, 85.7)
