File: layout/layout.kicad_sch (KiCad schematic)
At the start: 50 parts, among them J3 USB_C_Receptacle_USB2.0_16P, SW1 SW_Push, SW2 SW_Push, U1 AP2112K-3.3, U2 ESP32-S3-WROOM, U3 AL8860MP, U4 AL8860MP, U5 TPS54202DDC, U6 AL8860MP

Commit message: null
Parts:
- added J1: Conn_01x03_Socket, Connector_PinHeader_2.54mm:PinHeader_1x03_P2.54mm_Vertical, symbol Connector:Conn_01x03_Socket
- added J2: Conn_01x03_Pin, Connector_PinHeader_2.54mm:PinHeader_1x03_P2.54mm_Vertical, symbol Connector:Conn_01x03_Pin
- C10, C12, C14, C3, C4, C5, C6, C7, C8, C9: footprint Capacitor_SMD:C_0603_1608Metric -> Capacitor_SMD:C_0201_0603Metric
- D10, D2, D7: value RB070mm -> D0.7V; footprint Library:SODFL3617X108N -> Diode_SMD:D_0603_1608Metric
- D5, D6: value RB070mm -> D_Small; footprint Library:SODFL3617X108N -> Diode_SMD:D_0603_1608Metric
- R1, R10, R11, R12, R13, R14, R15, R16, R17, R2, R3, R4, R5, R6, R7, R8, R9: footprint Resistor_SMD:R_0603_1608Metric -> Resistor_SMD:R_0201_0603Metric
Connections:
- net GREEN_OUT is gone; now on net 3V1A: D4.2 (GK), L3.1
- net BLUE_OUT renamed 3V1A
- net DATA1: no longer names the net of R8.1
- net DATA1: now also J2.1 (Pin_1); no longer U2.36 (IO42)
- net DATA2: no longer names the net of U2.35 (IO41)
- net DATA2: now also J1.2 (Pin_2); no longer R11.1
- net DATA3: no longer names the net of U2.34 (IO40)
- net DATA3: now also J1.3 (Pin_3); no longer R9.1
- net RED_OUT renamed 2V1A
- new net: J1.1 (Pin_1), U2.36 (IO42)
- new net: J2.3 (Pin_3), R9.1
- new net: J2.2 (Pin_2), R11.1
